Commit message: updated URDF

File: Software/src/hexapod_description/urdf/hexapod.urdf.xacro (robot description, xacro)
@@ -75,5 +75,5 @@
     <link name="tibia_link_${side}${position}">
       <collision name="collision">
-        <origin rpy="0 0 0" xyz="0 0 0"/>
+        <origin rpy="0 ${pi} ${pi/2}" xyz="0 0 -0.0145"/>
         <!--<origin rpy="${pi} ${-pi/2} 0" xyz="0 0 0"/>-->
         <geometry>
