Commit message: revised_urdf

File: Software/src/hexapod_description_mk2/urdf/hexapod.urdf.xacro (robot description, xacro)
@@ -75,5 +75,5 @@
     <link name="tibia_link_${side}${position}">
       <collision name="collision">
-        <origin rpy="0 ${pi} ${pi/2}" xyz="0 0 -0.0145"/>
+        <origin rpy="0 ${pi} ${pi/2}" xyz="0 0 0"/>
         <!--<origin rpy="${pi} ${-pi/2} 0" xyz="0 0 0"/>-->
         <geometry>
@@ -83,5 +83,5 @@
       <visual name="visual">
         <!--<origin rpy="${pi} ${-pi/2} 0" xyz="0 0 0"/>-->
-        <origin rpy="0 ${pi} ${pi/2}" xyz="0 0 -0.0145"/>
+        <origin rpy="0 ${pi} ${pi/2}" xyz="0 0 0"/>
         <geometry>
           <mesh filename="package://hexapod_description_mk2/meshes/Tibia.dae"/>
@@ -90,5 +90,5 @@
     </link>
     <joint name="TIBIA_${side}${position}" type="revolute">
-      <origin rpy="0 0 0" xyz="0 ${femur_length} 0"/>
+      <origin rpy="0 0 0" xyz="0 ${femur_length} -0.0145"/>
       <child link="tibia_link_${side}${position}"/>
       <parent link="femur_link_${side}${position}"/>

Commit message: changed hexapod parameters
Simulation works

File: Software/src/hexapod_description_mk2/urdf/hexapod.urdf.xacro (robot description, xacro)
@@ -6,5 +6,5 @@
   <xacro:property name="femur_length" value="0.0645" />
   <xacro:property name="tibia_length" value="0.133" />
-  <xacro:property name="ground_offset" value="0.18" />
+  <xacro:property name="ground_offset" value="0.10" />
   <xacro:property name="offset_y_f" value="0.06091" />
   <xacro:property name="offset_y_r" value="0.06091" />
@@ -28,5 +28,5 @@
         <mesh filename="package://hexapod_description_mk2/meshes/Body.dae"/>
       </geometry>
-      <origin rpy="0 0 ${pi/2}" xyz="0.006985 0.0 ${ground_offset}"/>
+      <origin rpy="${pi} 0 ${3*pi/2}" xyz="0.006985 0.0 ${ground_offset}"/>
     </visual>
   </link>
@@ -40,5 +40,5 @@
         </geometry>
         <!--<origin rpy="0 ${pi/2} ${(1-axis)/2*pi}" xyz="0 ${axis*coxa_length} 0.024"/>-->
-        <origin rpy="0 ${pi/2} ${(2-axis)/2*pi}" xyz="0 0.0 0.0014"/>
+        <origin rpy="0 ${pi/2} ${(2-axis)/2*pi}" xyz="0 0.0 0.0"/>
       </visual>
     </link>
@@ -46,5 +46,5 @@
       <child link="coxa_link_${side}${position}"/>
       <parent link="base_link"/>
-      <origin rpy="0 0 ${angle}" xyz="${x} ${y} 0.194 "/>
+      <origin rpy="0 0 ${angle}" xyz="${x} ${y} ${ground_offset-0.015}"/>
       <axis xyz="0 0 ${-axis}"/>
       <limit effort="1000.0" lower="${-pi/2}" upper="${pi/2}" velocity="0.5"/>

Commit message: updated

File: Software/src/hexapod_description_mk2/urdf/hexapod.urdf.xacro (robot description, xacro)
@@ -58,5 +58,5 @@
       </collision>
       <visual name="visual">
-        <origin rpy="${pi/2} 0 ${3*pi/2}" xyz="0 0 0"/>
+        <origin rpy="${3*pi/2} 0 ${3*pi/2}" xyz="0 0 0"/>
         <!--<origin rpy="${pi/2} 0 ${axis*pi/2}" xyz="${axis*-0.024} ${femur_length/2} 0"/>-->
         <geometry>
